File: Picaxe 20X2 prop controller.kicad_sch (KiCad schematic)
At the start: 65 parts, among them J1 FC68131, J10 Conn_01x05_Male (- power bus), J11 Conn_01x08_Male - pin I/O, J12 MP3 player, J13 servo 2, J14 servo 3, J15 servo 4, J16 servo 5, J17 Ext servo power, J18 Servo power select, J19 C.0, J2 Conn_01x08_Male - pin I/O, J20 C.5, J21 C.1, J22 C.6, J23 C.2, J24 C.7, J25 C.3, J26 C.4, J27 B.6 TX, J28 OSTTC080162, J29 B.5 pin, J3 servo 1, J30 B.6, J31 I2C conn, J32 B.6, J33 Batt Connector, J34 Batt / Reg select, J4 servo 6, J5 B.7 RX, J6 OSTTC080162, J7 OSTTC020162, J8 PJ-202AH, J9 Conn_01x05_Male (+ power bus), U1 Picaxe 20X2, U3 L7805CV, U4 ULN2803A

Commit message: Board complete Beta test 1
Parts:
- added C7: .1uf, Capacitor_THT:C_Disc_D3.0mm_W2.0mm_P2.50mm, symbol Device:C_Small
- C3: footprint Capacitor_THT:CP_Radial_D5.0mm_P2.00mm -> Capacitor_THT:CP_Radial_D5.0mm_P2.50mm
- J30: value B.6 -> B.7
- J32: value B.6 -> B.5
- J34: value Batt / Reg select -> Batt in
Connections:
- net 5V: now also C7.1
- net GNDREF: now also C7.2
- net ob4: now also J29.2 (Pin_2)
- net ob5: no longer J29.2 (Pin_2)
Changed lines of the file:
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@@
+    (stroke (width 0) (type default) (color 0 0 0 0))
+  )
+  (wire (pts (xy 82.4992 41.3512) (xy 82.4992 42.4688))
     (stroke (width 0) (type default) (color 0 0 0 0))
   )
@@
     (effects (font (size 1.27 1.27)) (justify left bottom))
   )
-  (label "ob5" (at 49.7586 129.2606 0)
+  (label "ob4" (at 49.7586 129.2606 0)
     (effects (font (size 1.27 1.27)) (justify left bottom))
   )
   (label "ic0" (at 172.3644 120.777 0)
+    (effects (font (size 1.27 1.27)) (justify left bottom))
+  )
+  (label "5V" (at 82.4992 41.3512 0)
     (effects (font (size 1.27 1.27)) (justify left bottom))
   )
@@
     (in_bom yes) (on_board yes) (fields_autoplaced)
     (property "Reference" "J32" (id 0) (at 197.739 131.9022 0))
-    (property "Value" "B.6" (id 1) (at 197.739 134.4422 0)
+    (property "Value" "B.5" (id 1) (at 197.739 134.4422 0)
       (effects (font (size 1.27 1.27)) hide)
     )
@@
     (pin "2")
     (pin "3")
+  )
+  (symbol (lib_id "power:GNDREF") (at 82.4992 47.5488 0) (unit 1)
+    (in_bom yes) (on_board yes)
+    (property "Reference" "#PWR010" (id 0) (at 82.4992 53.8988 0)
+      (effects (font (size 1.27 1.27)) hide)
+    )
+    (property "Value" "GNDREF" (id 1) (at 82.4992 52.07 0))
+    (property "Footprint" "" (id 2) (at 82.4992 47.5488 0)
+      (effects (font (size 1.27 1.27)) hide)
+    )
+    (property "Datasheet" "" (id 3) (at 82.4992 47.5488 0)
+      (effects (font (size 1.27 1.27)) hide)
+    )
+    (pin "1")
   )
   (symbol (lib_id "Picaxe_Joe:Picaxe 20X2") (at 123.19 78.74 0) (unit 1)
@@
     (in_bom yes) (on_board yes)
     (property "Reference" "J34" (id 0) (at 15.1765 66.5099 90))
-    (property "Value" "Batt / Reg select" (id 1) (at 17.8435 65.9765 90))
+    (property "Value" "Batt in" (id 1) (at 17.8435 65.9765 90))
     (property "Footprint" "Connector_PinHeader_2.54mm:PinHeader_1x03_P2.54mm_Vertical" (id 2) (at 20.1168 66.548 0)
       (effects (font (size 1.27 1.27)) hide)
@@
     (in_bom yes) (on_board yes) (fields_autoplaced)
     (property "Reference" "J30" (id 0) (at 182.0164 131.8768 0))
-    (property "Value" "B.6" (id 1) (at 182.0164 134.4168 0)
+    (property "Value" "B.7" (id 1) (at 182.0164 134.4168 0)
       (effects (font (size 1.27 1.27)) hide)
     )
@@
     (pin "2")
   )
+  (symbol (lib_id "Device:C_Small") (at 82.4992 45.0088 0) (unit 1)
+    (in_bom yes) (on_board yes) (fields_autoplaced)
+    (property "Reference" "C7" (id 0) (at 85.4456 43.745 0)
+      (effects (font (size 1.27 1.27)) (justify left))
+    )
+    (property "Value" ".1uf" (id 1) (at 85.4456 46.285 0)
+      (effects (font (size 1.27 1.27)) (justify left))
+    )
+    (property "Footprint" "Capacitor_THT:C_Disc_D3.0mm_W2.0mm_P2.50mm" (id 2) (at 82.4992 45.0088 0)
+      (effects (font (size 1.27 1.27)) hide)
+    )
+    (property "Datasheet" "~" (id 3) (at 82.4992 45.0088 0)
+      (effects (font (size 1.27 1.27)) hide)
+    )
+    (pin "1")
+    (pin "2")
+  )
   (symbol (lib_id "power:GNDREF") (at 114.1222 173.2026 90) (unit 1)
     (in_bom yes) (on_board yes) (fields_autoplaced)
@@
       (effects (font (size 1.27 1.27)) (justify left))
     )
-    (property "Footprint" "Capacitor_THT:CP_Radial_D5.0mm_P2.00mm" (id 2) (at 84.2772 25.3492 0)
+    (property "Footprint" "Capacitor_THT:CP_Radial_D5.0mm_P2.50mm" (id 2) (at 84.2772 25.3492 0)
       (effects (font (size 1.27 1.27)) hide)
     )
@@
       (reference "#PWR09") (unit 1) (value "GNDREF") (footprint "")
     )
+    (path "/359f3573-b6ec-43ff-9e57-b7c42c9361c7"
+      (reference "#PWR010") (unit 1) (value "GNDREF") (footprint "")
+    )
     (path "/afcb086b-a91e-4c22-a67a-e2359a52cea8"
       (reference "#PWR0101") (unit 1) (value "GNDREF") (footprint "")
@@
     )
     (path "/ac69ac5b-2b9c-46b0-b895-b853d2f117d5"
-      (reference "C3") (unit 1) (value "10uf") (footprint "Capacitor_THT:CP_Radial_D5.0mm_P2.00mm")
+      (reference "C3") (unit 1) (value "10uf") (footprint "Capacitor_THT:CP_Radial_D5.0mm_P2.50mm")
     )
     (path "/de9f799c-f884-46f1-a6da-38bd6a3b44e1"
@@
       (reference "C6") (unit 1) (value ".1uf") (footprint "Capacitor_THT:C_Disc_D3.0mm_W2.0mm_P2.50mm")
     )
+    (path "/9900e5a4-c72d-4f78-8483-b605b0ecc497"
+      (reference "C7") (unit 1) (value ".1uf") (footprint "Capacitor_THT:C_Disc_D3.0mm_W2.0mm_P2.50mm")
+    )
     (path "/0c32625e-1c6d-476f-8155-56c1d4f91b84"
       (reference "D1") (unit 1) (value "LTL2R3KEK") (footprint "digikey-footprints:LED_5mm_Radial")
@@
     )
     (path "/83e53502-9510-4294-9334-311bd3dbe402"
-      (reference "J30") (unit 1) (value "B.6") (footprint "Connector_PinHeader_2.54mm:PinHeader_1x02_P2.54mm_Vertical")
+      (reference "J30") (unit 1) (value "B.7") (footprint "Connector_PinHeader_2.54mm:PinHeader_1x02_P2.54mm_Vertical")
     )
     (path "/9616e5c6-1c04-4885-98bc-59829af2252d"
@@
     )
     (path "/0bafae2e-441b-4483-84b4-f9087ac28dea"
-      (reference "J32") (unit 1) (value "B.6") (footprint "Connector_PinHeader_2.54mm:PinHeader_1x02_P2.54mm_Vertical")
+      (reference "J32") (unit 1) (value "B.5") (footprint "Connector_PinHeader_2.54mm:PinHeader_1x02_P2.54mm_Vertical")
     )
     (path "/8b60c28b-2164-4b2e-bb66-23cd9efd8df7"
@@
     )
     (path "/571822e8-0e38-4fc2-9bfc-81299bd0b279"
-      (reference "J34") (unit 1) (value "Batt / Reg select") (footprint "Connector_PinHeader_2.54mm:PinHeader_1x03_P2.54mm_Vertical")
+      (reference "J34") (unit 1) (value "Batt in") (footprint "Connector_PinHeader_2.54mm:PinHeader_1x03_P2.54mm_Vertical")
     )
     (path "/cd32adbb-b86c-4eee-aa17-84272d12d149"
